Commit message: ultrasone added to urdf

File: jvr_controller/urdf/jvr.urdf (robot description, URDF)
Before this commit: robot jvr, 2 links, 1 joints
Links:
- link ultrasone_sensor: geometry visual box size=0.005 0.043 0.02
Joints:
- joint joint_name: axis 0.0 1.0 0.0 -> 0.0 0.0 1.0; origin xyz=0.1 0.1 0.1 rpy=0.0 0.0 0.0 -> xyz=0.1 0.0 0.1 rpy=0.0 0.0 0.0

Commit message: sensor position adjusted

File: jvr_controller/urdf/jvr.urdf (robot description, URDF)
Before this commit: robot jvr, 2 links, 1 joints
Joints:
- joint joint_name: origin xyz=0.1 0.0 0.1 rpy=0.0 0.0 0.0 -> xyz=0.0765 0.0 0.08 rpy=0.0 0.0 0.0

Commit message: limits on servo set (-45 to +45 degrees)

File: jvr_controller/urdf/jvr.urdf (robot description, URDF)
Before this commit: robot jvr, 2 links, 1 joints
Joints:
- joint joint_name: limit lower=-1.0 upper=1.0 effort=0.0 velocity=0.0 -> lower=-0.785 upper=0.785 effort=0.0 velocity=0.0

Commit message: controller subscribed to objectdetected topic

File: jvr_controller/urdf/jvr.urdf (robot description, URDF)
Before this commit: robot jvr, 2 links, 1 joints
Joints:
- removed joint joint_name
- added joint SweepSensorServo: type revolute, parent chassis, child ultrasone_sensor, origin xyz=0.0765 0.0 0.08 rpy=0.0 0.0 0.0, axis 0.0 0.0 1.0, limit lower=-0.785 upper=0.785 effort=0.0 velocity=0.0

Commit message: servo moves "real time" and in correct rotation

File: jvr_controller/urdf/jvr.urdf (robot description, URDF)
Before this commit: robot jvr, 2 links, 1 joints
Joints:
- joint SweepSensorServo: axis 0.0 0.0 1.0 -> 0 0 1
