Commit message: urdf converted to xacro

File: description/jvr.robot.xacro (robot description, xacro)
@@ -1,4 +1,20 @@
 <?xml version="1.0"?>
-<robot name="jvr">
+<robot xmlns:xacro="http://www.ros.org/wiki/xacro" >
+    <!-- Materials -->
+    <material name="white">
+        <color rgba="1 1 1 1" />
+    </material>
+    <material name="orange">
+        <color rgba="1 0.3 0.1 1"/>
+    </material>
+    <material name="blue">
+        <color rgba="0.2 0.2 1 1"/>
+    </material>
+    <material name="black">
+        <color rgba="0 0 0 1"/>
+    </material>
+    <material name="yellow">
+        <color rgba="1 1 0 1"/>
+    </material>
     <!-- base (in middle of the two wheels) -->
     <link name="base_link">
@@ -13,10 +29,31 @@
     <link name="chassis">
         <visual>
-        <!-- <origin xyz="0.1025 0 0.015" /> -->
-        <origin xyz="0.1025 0 0.025" />
+            <!-- <origin xyz="0.1025 0 0.015" /> -->
+            <origin xyz="0.1025 0 0.025" />
             <geometry>
                 <box size="0.205 0.145 0.050" />
             </geometry>
+            <material name="black" />
         </visual>
+    </link>
+    <!-- Left wheel -->
+    <joint name="left_wheel_joint" type="continuous">
+        <parent link="base_link"/>
+        <child link="left_wheel"/>
+        <origin xyz="0 0.059 0" rpy="-${pi/2} 0 0" />
+        <axis xyz="0 0 1"/>
+    </joint>
+    <link name="left_wheel">
+        <visual>
+            <geometry>
+                <cylinder radius="0.05" length="0.04"/>
+            </geometry>
+            <material name="yellow"/>
+        </visual>
+        <collision>
+            <geometry>
+                <cylinder radius="0.05" length="0.04"/>
+            </geometry>
+        </collision>
     </link>
     <!-- <link name="chassis">

Commit message: both wheels and caster wheel

File: description/jvr.robot.xacro (robot description, xacro)
@@ -1,4 +1,4 @@
 <?xml version="1.0"?>
-<robot xmlns:xacro="http://www.ros.org/wiki/xacro" >
+<robot xmlns:xacro="http://www.ros.org/wiki/xacro">
     <!-- Materials -->
     <material name="white">
@@ -6,14 +6,17 @@
     </material>
     <material name="orange">
-        <color rgba="1 0.3 0.1 1"/>
+        <color rgba="1 0.3 0.1 1" />
     </material>
     <material name="blue">
-        <color rgba="0.2 0.2 1 1"/>
+        <color rgba="0.2 0.2 1 1" />
     </material>
     <material name="black">
-        <color rgba="0 0 0 1"/>
+        <color rgba="0 0 0 1" />
     </material>
     <material name="yellow">
-        <color rgba="1 1 0 1"/>
+        <color rgba="1 1 0 1" />
+    </material>
+    <material name="silver">
+        <color rgba="0.7 0.7 0.7 1" />
     </material>
     <!-- base (in middle of the two wheels) -->
@@ -23,11 +26,10 @@
     <!-- CHASSIS (simplified body of the jvr-robot) -->
     <joint name="chassis_joint" type="fixed">
-        <parent link="base_link"/>
-        <child link="chassis"/>
-        <origin xyz="-0.14 0 -0.015"/>
+        <parent link="base_link" />
+        <child link="chassis" />
+        <origin xyz="-0.14 0 -0.015" />
     </joint>
     <link name="chassis">
         <visual>
-            <!-- <origin xyz="0.1025 0 0.015" /> -->
             <origin xyz="0.1025 0 0.025" />
             <geometry>
@@ -38,61 +40,63 @@
     </link>
     <!-- Left wheel -->
+    <!-- The weels are half inside the box, because the outer edges are used as chassis -->
     <joint name="left_wheel_joint" type="continuous">
-        <parent link="base_link"/>
-        <child link="left_wheel"/>
-        <origin xyz="0 0.059 0" rpy="-${pi/2} 0 0" />
-        <axis xyz="0 0 1"/>
+        <parent link="base_link" />
+        <child link="left_wheel" />
+        <origin xyz="0 0.072 0" rpy="-${pi/2} 0 0" />
+        <axis xyz="0 0 1" />
     </joint>
     <link name="left_wheel">
         <visual>
             <geometry>
-                <cylinder radius="0.05" length="0.04"/>
+                <cylinder radius="0.05" length="0.026" />
             </geometry>
-            <material name="yellow"/>
+            <material name="yellow" />
         </visual>
         <collision>
             <geometry>
-                <cylinder radius="0.05" length="0.04"/>
+                <cylinder radius="0.05" length="0.04" />
             </geometry>
         </collision>
     </link>
-    <!-- <link name="chassis">
-        <visual name="bottom_plate">
-            <origin xyz="0.0 0.0 0.013" rpy="0.0 0.0 0.0"/>
+    <!-- Right wheel -->
+    <!-- The weels are half inside the box, because the outer edges are used as chassis -->
+    <joint name="right_wheel_joint" type="continuous">
+        <parent link="base_link" />
+        <child link="right_wheel" />
+        <origin xyz="0 -0.072 0" rpy="${pi/2} 0 0" />
+        <axis xyz="0 0 -1" />
+    </joint>
+    <link name="right_wheel">
+        <visual>
             <geometry>
-                <box size="0.195 0.103 0.005"/>
+                <cylinder radius="0.05" length="0.026" />
             </geometry>
-            <material name="black">
-                <color rgba="0.9 0.9 0.9 1.0"/>
-            </material>
+            <material name="yellow" />
         </visual>
-        <visual name="top_plate">
-            <origin xyz="0.0 0.0 0.060" rpy="0.0 0.0 0.0"/>
+        <collision>
             <geometry>
-                <box size="0.195 0.103 0.005"/>
+                <cylinder radius="0.05" length="0.04" />
             </geometry>
-            <material name="black">
-                <color rgba="0.7 0.7 0.7 1.0"/>
-            </material>
+        </collision>
+    </link>
+    <!-- Caster 1.6 -->
+    <joint name="caster_wheel_joint" type="fixed">
+        <parent link="chassis"/>
+        <child link="caster_wheel"/>
+        <origin xyz="0.016 0 -0.015"/>
+    </joint>
+    <link name="caster_wheel">
+        <visual>
+            <geometry>
+                <sphere radius="0.008"/>
+            </geometry>
+            <material name="silver"/>
         </visual>
+        <collision>
+            <geometry>
+                <sphere radius="0.008"/>
+            </geometry>
+        </collision>
     </link>
-    <link name="ultrasone_sensor">
-        <visual name="">
-            <origin xyz="0.0 0.0 0.0" rpy="0.0 0.0 0.0"/>
-            <geometry>
-                <box size="0.005 0.043 0.02"/>
-            </geometry>
-            <material name="blue">
-                <color rgba="0.0 1.0 0.0 1.0"/>
-                <texture filename=""/>
-            </material>
-        </visual>
-    </link>
-	<joint name="SweepSensorServo" type="revolute">
-        <origin xyz="0.0765 0.0 0.08" rpy="0.0 0.0 0.0"/>
-        <parent link="chassis"/>
-        <child link="ultrasone_sensor"/>
-        <axis xyz="0 0 1"/>
-        <limit lower="-0.785" upper="0.785" effort="0.0" velocity="0.0"/>
-    </joint> -->
 </robot>

Commit message: spaces removed

File: description/jvr.robot.xacro (robot description, xacro)
@@ -3,38 +3,38 @@
     <!-- Materials -->
     <material name="white">
-        <color rgba="1 1 1 1" />
+        <color rgba="1 1 1 1"/>
     </material>
     <material name="orange">
-        <color rgba="1 0.3 0.1 1" />
+        <color rgba="1 0.3 0.1 1"/>
     </material>
     <material name="blue">
-        <color rgba="0.2 0.2 1 1" />
+        <color rgba="0.2 0.2 1 1"/>
     </material>
     <material name="black">
-        <color rgba="0 0 0 1" />
+        <color rgba="0 0 0 1"/>
     </material>
     <material name="yellow">
-        <color rgba="1 1 0 1" />
+        <color rgba="1 1 0 1"/>
     </material>
     <material name="silver">
-        <color rgba="0.7 0.7 0.7 1" />
+        <color rgba="0.7 0.7 0.7 1"/>
     </material>
     <!-- base (in middle of the two wheels) -->
     <link name="base_link">
-        <origin xyz="0 0 0.033" />
+        <origin xyz="0 0 0.033"/>
     </link>
     <!-- CHASSIS (simplified body of the jvr-robot) -->
     <joint name="chassis_joint" type="fixed">
-        <parent link="base_link" />
-        <child link="chassis" />
-        <origin xyz="-0.14 0 -0.015" />
+        <parent link="base_link"/>
+        <child link="chassis"/>
+        <origin xyz="-0.14 0 -0.015"/>
     </joint>
     <link name="chassis">
         <visual>
-            <origin xyz="0.1025 0 0.025" />
+            <origin xyz="0.1025 0 0.025"/>
             <geometry>
-                <box size="0.205 0.145 0.050" />
+                <box size="0.205 0.145 0.050"/>
             </geometry>
-            <material name="black" />
+            <material name="black"/>
         </visual>
     </link>
@@ -42,19 +42,19 @@
     <!-- The weels are half inside the box, because the outer edges are used as chassis -->
     <joint name="left_wheel_joint" type="continuous">
-        <parent link="base_link" />
-        <child link="left_wheel" />
-        <origin xyz="0 0.072 0" rpy="-${pi/2} 0 0" />
-        <axis xyz="0 0 1" />
+        <parent link="base_link"/>
+        <child link="left_wheel"/>
+        <origin xyz="0 0.072 0" rpy="-${pi/2} 0 0"/>
+        <axis xyz="0 0 1"/>
     </joint>
     <link name="left_wheel">
         <visual>
             <geometry>
-                <cylinder radius="0.05" length="0.026" />
+                <cylinder radius="0.05" length="0.026"/>
             </geometry>
-            <material name="yellow" />
+            <material name="yellow"/>
         </visual>
         <collision>
             <geometry>
-                <cylinder radius="0.05" length="0.04" />
+                <cylinder radius="0.05" length="0.04"/>
             </geometry>
         </collision>
@@ -63,19 +63,19 @@
     <!-- The weels are half inside the box, because the outer edges are used as chassis -->
     <joint name="right_wheel_joint" type="continuous">
-        <parent link="base_link" />
-        <child link="right_wheel" />
-        <origin xyz="0 -0.072 0" rpy="${pi/2} 0 0" />
-        <axis xyz="0 0 -1" />
+        <parent link="base_link"/>
+        <child link="right_wheel"/>
+        <origin xyz="0 -0.072 0" rpy="${pi/2} 0 0"/>
+        <axis xyz="0 0 -1"/>
     </joint>
     <link name="right_wheel">
         <visual>
             <geometry>
-                <cylinder radius="0.05" length="0.026" />
+                <cylinder radius="0.05" length="0.026"/>
             </geometry>
-            <material name="yellow" />
+            <material name="yellow"/>
         </visual>
         <collision>
             <geometry>
-                <cylinder radius="0.05" length="0.04" />
+                <cylinder radius="0.05" length="0.04"/>
             </geometry>
         </collision>

Commit message: sweep sensor (joint and backplate)

File: description/jvr.robot.xacro (robot description, xacro)
@@ -100,3 +100,25 @@
         </collision>
     </link>
+    <!-- Sweep sensor -->
+    <joint name="sweep_sensor_joint" type="revolute">
+        <parent link="chassis"/>
+        <child link="sweep_sensor"/>
+        <origin xyz="0.175 0 0.059"/>
+        <axis xyz="0 0 1"/>
+        <limit lower="-${(pi/180)*45}" upper="${(pi/180)*45}" effort="100.0" velocity="${((pi/180)*60)/0.3}"/> <!-- not sure what 'effort' means -->
+    </joint>
+    <link name="sweep_sensor">
+        <visual>
+            <origin xyz="0.009 0 0.018"/>
+            <geometry>
+                <box size="0.002 0.05 0.036"/>
+            </geometry>
+            <material name="blue"/>
+        </visual>
+        <collision>
+            <geometry>
+                <box size="0.002 0.05 0.036"/>
+            </geometry>
+        </collision>
+    </link>
 </robot>

Commit message: documentation added

File: description/jvr.robot.xacro (robot description, xacro)
@@ -106,5 +106,8 @@
         <origin xyz="0.175 0 0.059"/>
         <axis xyz="0 0 1"/>
-        <limit lower="-${(pi/180)*45}" upper="${(pi/180)*45}" effort="100.0" velocity="${((pi/180)*60)/0.3}"/> <!-- not sure what 'effort' means -->
+        <!-- lower limit -45deg, upper limit 45deg-->
+        <!-- not sure what 'effort' means -->
+        <!-- speed 60 deg per 0.3 secs. see https://osoyoo.store/en-eu/products/micro-servo-sg90-blue-for-arduino-v2-0-robot-carmodel-lacc200610#tab_technical-details -->
+        <limit lower="-${(pi/180)*45}" upper="${(pi/180)*45}" effort="100.0" velocity="${((pi/180)*60)/0.3}"/>
     </joint>
     <link name="sweep_sensor">

Commit message: sweep sensor added

File: description/jvr.robot.xacro (robot description, xacro)
@@ -56,5 +56,5 @@
         <collision>
             <geometry>
-                <cylinder radius="0.05" length="0.04"/>
+                <cylinder radius="0.05" length="0.026"/>
             </geometry>
         </collision>
@@ -77,5 +77,5 @@
         <collision>
             <geometry>
-                <cylinder radius="0.05" length="0.04"/>
+                <cylinder radius="0.05" length="0.026"/>
             </geometry>
         </collision>
@@ -104,5 +104,5 @@
         <parent link="chassis"/>
         <child link="sweep_sensor"/>
-        <origin xyz="0.175 0 0.059"/>
+        <origin xyz="0.187 0 0.059"/>
         <axis xyz="0 0 1"/>
         <!-- lower limit -45deg, upper limit 45deg-->
@@ -117,9 +117,24 @@
                 <box size="0.002 0.05 0.036"/>
             </geometry>
-            <material name="blue"/>
+            <material name="silver"/>
+        </visual>
+        <visual>
+            <origin xyz="0.015 0.01 0.018" rpy="0 ${pi/2} 0"/>
+            <geometry>
+                <cylinder radius="0.008" length="0.01"/>
+            </geometry>
+            <material name="silver"/>
+        </visual>
+        <visual>
+            <origin xyz="0.015 -0.01 0.018" rpy="0 ${pi/2} 0"/>
+            <geometry>
+                <cylinder radius="0.008" length="0.01"/>
+            </geometry>
+            <material name="silver"/>
         </visual>
         <collision>
+        <origin xyz="0.009 0 0.018"/>
             <geometry>
-                <box size="0.002 0.05 0.036"/>
+                <box size="0.014 0.05 0.036"/>
             </geometry>
         </collision>

Commit message: collision of chassis

File: description/jvr.robot.xacro (robot description, xacro)
@@ -38,4 +38,10 @@
             <material name="black"/>
         </visual>
+        <collision>
+            <origin xyz="0.1025 0 0.025"/>
+            <geometry>
+                <box size="0.205 0.145 0.050"/>
+            </geometry>
+        </collision>
     </link>
     <!-- Left wheel -->
@@ -134,5 +140,5 @@
         </visual>
         <collision>
-        <origin xyz="0.009 0 0.018"/>
+            <origin xyz="0.009 0 0.018"/>
             <geometry>
                 <box size="0.014 0.05 0.036"/>
