Commit message: Inertia added

File: description/jvr.robot.xacro (robot description, xacro)
@@ -1,4 +1,49 @@
 <?xml version="1.0"?>
 <robot xmlns:xacro="http://www.ros.org/wiki/xacro">
+    <xacro:include filename="inertial_macros.xacro"/>
+    <!-- Dimensions -->
+    <!-- Chassis -->
+    <xacro:property name="chassis_length" value="0.205"/>
+    <xacro:property name="chassis_width" value="0.145"/>
+    <xacro:property name="chassis_height" value="0.050"/>
+    <xacro:property name="chassis_mass" value="0.6"/>
+    <!-- Wheels -->
+    <xacro:property name="wheel_radius" value="0.05"/>
+    <xacro:property name="wheel_thickness" value="0.026"/>
+    <xacro:property name="wheel_mass" value="0.038"/>
+    <xacro:property name="wheel_offset_x" value="0.14"/>
+    <xacro:property name="wheel_offset_y" value="0.072"/>
+    <xacro:property name="wheel_offset_z" value="0.015"/>
+    <!-- Caster wheel -->
+    <xacro:property name="caster_wheel_radius" value="0.008"/>
+    <xacro:property name="caster_wheel_mass" value="0.016"/>
+    <xacro:property name="caster_wheel_offset_x" value="0.016"/>
+    <xacro:property name="caster_wheel_offset_z" value="-0.015"/>
+    <!-- Sweep sensor -->
+    <xacro:property name="sweep_sensor_joint_offset_x" value="0.187"/>
+    <xacro:property name="sweep_sensor_joint_offset_z" value="0.059"/>
+    <!-- lower limit -45deg, upper limit 45deg-->
+    <!-- not sure what 'effort' means -->
+    <!-- speed 60 deg per 0.3 secs. see https://osoyoo.store/en-eu/products/micro-servo-sg90-blue-for-arduino-v2-0-robot-carmodel-lacc200610#tab_technical-details -->
+    <xacro:property name="sweep_sensor_joint_lower" value="-${(pi/180)*45}"/>
+    <xacro:property name="sweep_sensor_joint_upper" value="${(pi/180)*45}"/>
+    <xacro:property name="sweep_sensor_joint_effort" value="100.0"/>
+    <xacro:property name="sweep_sensor_joint_velocity" value="${((pi/180)*60)/0.3}"/>
+    <xacro:property name="sweep_sensor_mass" value="0.015"/>
+    <xacro:property name="sweep_sensor_backplate_offset_x" value="0.009"/>
+    <xacro:property name="sweep_sensor_backplate_offset_z" value="0.018"/>
+    <xacro:property name="sweep_sensor_backplate_length" value="0.002"/>
+    <xacro:property name="sweep_sensor_backplate_width" value="0.050"/>
+    <xacro:property name="sweep_sensor_backplate_height" value="0.036"/>
+    <xacro:property name="sweep_sensor_mic_offset_x" value="0.015"/>
+    <xacro:property name="sweep_sensor_mic_offset_y" value="0.010"/>
+    <xacro:property name="sweep_sensor_mic_offset_z" value="0.018"/>
+    <xacro:property name="sweep_sensor_mic_radius" value="0.008"/>
+    <xacro:property name="sweep_sensor_mic_length" value="0.010"/>
+    <xacro:property name="sweep_sensor_collision_length" value="${sweep_sensor_backplate_length + sweep_sensor_mic_length}"/>
+    <xacro:property name="sweep_sensor_collision_width" value="${sweep_sensor_backplate_width}"/>
+    <xacro:property name="sweep_sensor_collision_height" value="${sweep_sensor_backplate_height}"/>
+    <xacro:property name="sweep_sensor_collision_offset_x" value="${sweep_sensor_backplate_offset_x + (sweep_sensor_collision_length/2)}"/>
+    <xacro:property name="sweep_sensor_collision_offset_z" value="${sweep_sensor_backplate_offset_z}"/>
     <!-- Materials -->
     <material name="white">
@@ -28,20 +73,23 @@
         <parent link="base_link"/>
         <child link="chassis"/>
-        <origin xyz="-0.14 0 -0.015"/>
+        <origin xyz="${-wheel_offset_x} 0 ${-wheel_offset_z}"/>
     </joint>
     <link name="chassis">
         <visual>
-            <origin xyz="0.1025 0 0.025"/>
-            <geometry>
-                <box size="0.205 0.145 0.050"/>
+            <origin xyz="${chassis_length/2} 0 ${chassis_height/2}"/>
+            <geometry>
+                <box size="${chassis_length} ${chassis_width} ${chassis_height}"/>
             </geometry>
             <material name="black"/>
         </visual>
         <collision>
-            <origin xyz="0.1025 0 0.025"/>
-            <geometry>
-                <box size="0.205 0.145 0.050"/>
-            </geometry>
-        </collision>
+            <origin xyz="${chassis_length/2} 0 ${chassis_height/2}"/>
+            <geometry>
+                <box size="${chassis_length} ${chassis_width} ${chassis_height}"/>
+            </geometry>
+        </collision>
+        <xacro:inertial_box mass="${chassis_mass}" x="${chassis_length}" y="${chassis_width}" z="${chassis_height}">
+            <origin xyz="${chassis_length/2} 0 ${chassis_height/2}" rpy="0 0 0"/>
+        </xacro:inertial_box>
     </link>
     <!-- Left wheel -->
@@ -50,19 +98,24 @@
         <parent link="base_link"/>
         <child link="left_wheel"/>
-        <origin xyz="0 0.072 0" rpy="-${pi/2} 0 0"/>
+        <origin xyz="0 ${wheel_offset_y} 0" rpy="-${pi/2} 0 0"/>
         <axis xyz="0 0 1"/>
     </joint>
     <link name="left_wheel">
         <visual>
-            <geometry>
-                <cylinder radius="0.05" length="0.026"/>
+            <origin xyz="0 0 0" rpy="0 0 0"/>
+            <geometry>
+                <cylinder radius="${wheel_radius}" length="${wheel_thickness}"/>
             </geometry>
             <material name="yellow"/>
         </visual>
         <collision>
-            <geometry>
-                <cylinder radius="0.05" length="0.026"/>
-            </geometry>
-        </collision>
+            <origin xyz="0 0 0" rpy="0 0 0"/>
+            <geometry>
+                <cylinder radius="${wheel_radius}" length="${wheel_thickness}"/>
+            </geometry>
+        </collision>
+        <xacro:inertial_cylinder mass="${wheel_mass}" length="${wheel_thickness}" radius="${wheel_radius}">
+            <origin xyz="0 0 0" rpy="0 0 0"/>
+        </xacro:inertial_cylinder>
     </link>
     <!-- Right wheel -->
@@ -71,19 +124,24 @@
         <parent link="base_link"/>
         <child link="right_wheel"/>
-        <origin xyz="0 -0.072 0" rpy="${pi/2} 0 0"/>
+        <origin xyz="0 ${-wheel_offset_y} 0" rpy="${pi/2} 0 0"/>
         <axis xyz="0 0 -1"/>
     </joint>
     <link name="right_wheel">
         <visual>
-            <geometry>
-                <cylinder radius="0.05" length="0.026"/>
+            <origin xyz="0 0 0" rpy="0 0 0"/>
+            <geometry>
+                <cylinder radius="${wheel_radius}" length="${wheel_thickness}"/>
             </geometry>
             <material name="yellow"/>
         </visual>
         <collision>
-            <geometry>
-                <cylinder radius="0.05" length="0.026"/>
-            </geometry>
-        </collision>
+            <origin xyz="0 0 0" rpy="0 0 0"/>
+            <geometry>
+                <cylinder radius="${wheel_radius}" length="${wheel_thickness}"/>
+            </geometry>
+        </collision>
+        <xacro:inertial_cylinder mass="${wheel_mass}" length="${wheel_thickness}" radius="${wheel_radius}">
+            <origin xyz="0 0 0" rpy="0 0 0"/>
+        </xacro:inertial_cylinder>
     </link>
     <!-- Caster wheel -->
@@ -91,18 +149,23 @@
         <parent link="chassis"/>
         <child link="caster_wheel"/>
-        <origin xyz="0.016 0 -0.015"/>
+        <origin xyz="${caster_wheel_offset_x} 0 ${caster_wheel_offset_z}"/>
     </joint>
     <link name="caster_wheel">
         <visual>
-            <geometry>
-                <sphere radius="0.008"/>
-            </geometry>
-            <material name="silver"/>
-        </visual>
-        <collision>
-            <geometry>
-                <sphere radius="0.008"/>
-            </geometry>
-        </collision>
+            <origin xyz="0 0 0" rpy="0 0 0"/>
+            <geometry>
+                <sphere radius="${caster_wheel_radius}"/>
+            </geometry>
+            <material name="silver"/>
+        </visual>
+        <collision>
+            <origin xyz="0 0 0" rpy="0 0 0"/>
+            <geometry>
+                <sphere radius="${caster_wheel_radius}"/>
+            </geometry>
+        </collision>
+        <xacro:inertial_sphere mass="${caster_wheel_mass}" radius="${caster_wheel_radius}">
+            <origin xyz="0 0 0" rpy="0 0 0"/>
+        </xacro:inertial_sphere>
     </link>
     <!-- Sweep sensor -->
@@ -110,39 +173,40 @@
         <parent link="chassis"/>
         <child link="sweep_sensor"/>
-        <origin xyz="0.187 0 0.059"/>
+        <origin xyz="${sweep_sensor_joint_offset_x} 0 ${sweep_sensor_joint_offset_z}"/>
         <axis xyz="0 0 1"/>
-        <!-- lower limit -45deg, upper limit 45deg-->
-        <!-- not sure what 'effort' means -->
-        <!-- speed 60 deg per 0.3 secs. see https://osoyoo.store/en-eu/products/micro-servo-sg90-blue-for-arduino-v2-0-robot-carmodel-lacc200610#tab_technical-details -->
-        <limit lower="-${(pi/180)*45}" upper="${(pi/180)*45}" effort="100.0" velocity="${((pi/180)*60)/0.3}"/>
+        <limit lower="${sweep_sensor_joint_lower}" upper="${sweep_sensor_joint_upper}" effort="${sweep_sensor_joint_effort}" velocity="${sweep_sensor_joint_velocity}"/>
     </joint>
     <link name="sweep_sensor">
         <visual>
-            <origin xyz="0.009 0 0.018"/>
-            <geometry>
-                <box size="0.002 0.05 0.036"/>
-            </geometry>
-            <material name="silver"/>
-        </visual>
-        <visual>
-            <origin xyz="0.015 0.01 0.018" rpy="0 ${pi/2} 0"/>
-            <geometry>
-                <cylinder radius="0.008" length="0.01"/>
-            </geometry>
-            <material name="silver"/>
-        </visual>
-        <visual>
-            <origin xyz="0.015 -0.01 0.018" rpy="0 ${pi/2} 0"/>
-            <geometry>
-                <cylinder radius="0.008" length="0.01"/>
-            </geometry>
-            <material name="silver"/>
-        </visual>
-        <collision>
-            <origin xyz="0.009 0 0.018"/>
-            <geometry>
-                <box size="0.014 0.05 0.036"/>
-            </geometry>
-        </collision>
+            <origin xyz="${sweep_sensor_backplate_offset_x} 0 ${sweep_sensor_backplate_offset_z}"/>
+            <geometry>
+                <box size="${sweep_sensor_backplate_length} ${sweep_sensor_backplate_width} ${sweep_sensor_backplate_height}"/>
+            </geometry>
+            <material name="silver"/>
+        </visual>
+        <visual>
+            <origin xyz="${sweep_sensor_mic_offset_x} ${sweep_sensor_mic_offset_z} ${sweep_sensor_mic_offset_z}" rpy="0 ${pi/2} 0"/>
+            <geometry>
+                <cylinder radius="${sweep_sensor_mic_radius}" length="${sweep_sensor_mic_length}"/>
+            </geometry>
+            <material name="silver"/>
+        </visual>
+        <visual>
+            <origin xyz="${sweep_sensor_mic_offset_x} ${-sweep_sensor_mic_offset_z} ${sweep_sensor_mic_offset_z}" rpy="0 ${pi/2} 0"/>
+            <geometry>
+                <cylinder radius="${sweep_sensor_mic_radius}" length="${sweep_sensor_mic_length}"/>
+            </geometry>
+            <material name="silver"/>
+        </visual>
+        <collision>
+            <origin xyz="${sweep_sensor_collision_offset_x} 0 ${sweep_sensor_collision_offset_z}"/>
+            <geometry>
+                <box size="${sweep_sensor_collision_length} ${sweep_sensor_collision_width} ${sweep_sensor_collision_height}"/>
+            </geometry>
+        </collision>
+        <!-- using collision box for inertia-->
+        <xacro:inertial_box mass="${sweep_sensor_mass}" x="${sweep_sensor_collision_length}" y="${sweep_sensor_collision_width}" z="${sweep_sensor_collision_height}">
+            <origin xyz="${sweep_sensor_collision_offset_x} 0 ${sweep_sensor_collision_offset_z}" rpy="0 0 0"/>
+        </xacro:inertial_box>
     </link>
 </robot>

Commit message: some minor measurement changes

File: description/jvr.robot.xacro (robot description, xacro)
@@ -9,15 +9,15 @@
     <xacro:property name="chassis_mass" value="0.6"/>
     <!-- Wheels -->
-    <xacro:property name="wheel_radius" value="0.05"/>
+    <xacro:property name="wheel_radius" value="0.033"/>
     <xacro:property name="wheel_thickness" value="0.026"/>
     <xacro:property name="wheel_mass" value="0.038"/>
     <xacro:property name="wheel_offset_x" value="0.14"/>
     <xacro:property name="wheel_offset_y" value="0.072"/>
-    <xacro:property name="wheel_offset_z" value="0.015"/>
+    <xacro:property name="wheel_offset_z" value="0.014"/>
     <!-- Caster wheel -->
     <xacro:property name="caster_wheel_radius" value="0.008"/>
     <xacro:property name="caster_wheel_mass" value="0.016"/>
     <xacro:property name="caster_wheel_offset_x" value="0.016"/>
-    <xacro:property name="caster_wheel_offset_z" value="-0.015"/>
+    <xacro:property name="caster_wheel_offset_z" value="-0.012"/>
     <!-- Sweep sensor -->
     <xacro:property name="sweep_sensor_joint_offset_x" value="0.187"/>

Commit message: it should drive now

File: description/jvr.robot.xacro (robot description, xacro)
@@ -15,4 +15,5 @@
     <xacro:property name="wheel_offset_y" value="0.072"/>
     <xacro:property name="wheel_offset_z" value="0.014"/>
+    <xacro:property name="wheel_separation" value="${2 * wheel_offset_y}"/>
     <!-- Caster wheel -->
     <xacro:property name="caster_wheel_radius" value="0.008"/>
@@ -210,3 +211,14 @@
         </xacro:inertial_box>
     </link>
+    <gazebo>
+        <!--diff drive plugin-->
+        <plugin filename="gz-sim-diff-drive-system" name="gz::sim::systems::DiffDrive">
+            <left_joint>left_wheel_joint</left_joint>
+            <right_joint>right_wheel_joint</right_joint>
+            <wheel_separation>${wheel_separation}</wheel_separation>
+            <wheel_radius>${wheel_radius}</wheel_radius>
+            <odom_publish_frequency>1</odom_publish_frequency>
+            <topic>cmd_vel</topic>
+        </plugin>
+    </gazebo>
 </robot>
