Commit message: bridge tussen gazebo en ros2

File: description/jvr.robot.xacro (robot description, xacro)
@@ -43,12 +43,9 @@
     <xacro:property name="sweep_sensor_mic_radius" value="0.008" />
     <xacro:property name="sweep_sensor_mic_length" value="0.010" />
-    <xacro:property name="sweep_sensor_collision_length"
-        value="${sweep_sensor_backplate_length + sweep_sensor_mic_length}" />
+    <xacro:property name="sweep_sensor_collision_length" value="${sweep_sensor_backplate_length + sweep_sensor_mic_length}" />
     <xacro:property name="sweep_sensor_collision_width" value="${sweep_sensor_backplate_width}" />
     <xacro:property name="sweep_sensor_collision_height" value="${sweep_sensor_backplate_height}" />
-    <xacro:property name="sweep_sensor_collision_offset_x"
-        value="${sweep_sensor_backplate_offset_x + (sweep_sensor_collision_length/2)}" />
-    <xacro:property name="sweep_sensor_collision_offset_z"
-        value="${sweep_sensor_backplate_offset_z}" />
+    <xacro:property name="sweep_sensor_collision_offset_x" value="${sweep_sensor_backplate_offset_x + (sweep_sensor_collision_length/2)}" />
+    <xacro:property name="sweep_sensor_collision_offset_z" value="${sweep_sensor_backplate_offset_z}" />
     <!-- Materials -->
     <material name="white">
@@ -94,6 +91,5 @@
             </geometry>
         </collision>
-        <xacro:inertial_box mass="${chassis_mass}" x="${chassis_length}" y="${chassis_width}"
-            z="${chassis_height}">
+        <xacro:inertial_box mass="${chassis_mass}" x="${chassis_length}" y="${chassis_width}" z="${chassis_height}">
             <origin xyz="${chassis_length/2} 0 ${chassis_height/2}" rpy="0 0 0" />
         </xacro:inertial_box>
@@ -121,6 +117,5 @@
             </geometry>
         </collision>
-        <xacro:inertial_cylinder mass="${wheel_mass}" length="${wheel_thickness}"
-            radius="${wheel_radius}">
+        <xacro:inertial_cylinder mass="${wheel_mass}" length="${wheel_thickness}" radius="${wheel_radius}">
             <origin xyz="0 0 0" rpy="0 0 0" />
         </xacro:inertial_cylinder>
@@ -148,6 +143,5 @@
             </geometry>
         </collision>
-        <xacro:inertial_cylinder mass="${wheel_mass}" length="${wheel_thickness}"
-            radius="${wheel_radius}">
+        <xacro:inertial_cylinder mass="${wheel_mass}" length="${wheel_thickness}" radius="${wheel_radius}">
             <origin xyz="0 0 0" rpy="0 0 0" />
         </xacro:inertial_cylinder>
@@ -183,6 +177,5 @@
         <origin xyz="${sweep_sensor_joint_offset_x} 0 ${sweep_sensor_joint_offset_z}" />
         <axis xyz="0 0 1" />
-        <limit lower="${sweep_sensor_joint_lower}" upper="${sweep_sensor_joint_upper}"
-            effort="${sweep_sensor_joint_effort}" velocity="${sweep_sensor_joint_velocity}" />
+        <limit lower="${sweep_sensor_joint_lower}" upper="${sweep_sensor_joint_upper}" effort="${sweep_sensor_joint_effort}" velocity="${sweep_sensor_joint_velocity}" />
     </joint>
     <link name="sweep_sensor">
@@ -190,13 +183,10 @@
             <origin xyz="${sweep_sensor_backplate_offset_x} 0 ${sweep_sensor_backplate_offset_z}" />
             <geometry>
-                <box
-                    size="${sweep_sensor_backplate_length} ${sweep_sensor_backplate_width} ${sweep_sensor_backplate_height}" />
-            </geometry>
-            <material name="silver" />
-        </visual>
-        <visual>
-            <origin
-                xyz="${sweep_sensor_mic_offset_x} ${sweep_sensor_mic_offset_z} ${sweep_sensor_mic_offset_z}"
-                rpy="0 ${pi/2} 0" />
+                <box size="${sweep_sensor_backplate_length} ${sweep_sensor_backplate_width} ${sweep_sensor_backplate_height}" />
+            </geometry>
+            <material name="silver" />
+        </visual>
+        <visual>
+            <origin xyz="${sweep_sensor_mic_offset_x} ${sweep_sensor_mic_offset_z} ${sweep_sensor_mic_offset_z}" rpy="0 ${pi/2} 0" />
             <geometry>
                 <cylinder radius="${sweep_sensor_mic_radius}" length="${sweep_sensor_mic_length}" />
@@ -205,7 +195,5 @@
         </visual>
         <visual>
-            <origin
-                xyz="${sweep_sensor_mic_offset_x} ${-sweep_sensor_mic_offset_z} ${sweep_sensor_mic_offset_z}"
-                rpy="0 ${pi/2} 0" />
+            <origin xyz="${sweep_sensor_mic_offset_x} ${-sweep_sensor_mic_offset_z} ${sweep_sensor_mic_offset_z}" rpy="0 ${pi/2} 0" />
             <geometry>
                 <cylinder radius="${sweep_sensor_mic_radius}" length="${sweep_sensor_mic_length}" />
@@ -216,13 +204,10 @@
             <origin xyz="${sweep_sensor_collision_offset_x} 0 ${sweep_sensor_collision_offset_z}" />
             <geometry>
-                <box
-                    size="${sweep_sensor_collision_length} ${sweep_sensor_collision_width} ${sweep_sensor_collision_height}" />
+                <box size="${sweep_sensor_collision_length} ${sweep_sensor_collision_width} ${sweep_sensor_collision_height}" />
             </geometry>
         </collision>
         <!-- using collision box for inertia-->
-        <xacro:inertial_box mass="${sweep_sensor_mass}" x="${sweep_sensor_collision_length}"
-            y="${sweep_sensor_collision_width}" z="${sweep_sensor_collision_height}">
-            <origin xyz="${sweep_sensor_collision_offset_x} 0 ${sweep_sensor_collision_offset_z}"
-                rpy="0 0 0" />
+        <xacro:inertial_box mass="${sweep_sensor_mass}" x="${sweep_sensor_collision_length}" y="${sweep_sensor_collision_width}" z="${sweep_sensor_collision_height}">
+            <origin xyz="${sweep_sensor_collision_offset_x} 0 ${sweep_sensor_collision_offset_z}" rpy="0 0 0" />
         </xacro:inertial_box>
     </link>
@@ -237,4 +222,9 @@
             <!-- <topic>cmd_vel</topic> -->
         </plugin>
+        <plugin filename="ignition-gazebo-joint-state-publisher-system" name="ignition::gazebo::systems::JointStatePublisher" />
+        <plugin filename="ignition-gazebo-pose-publisher-system" name="ignition::gazebo::systems::PosePublisher">
+            <publish_link_pose>true</publish_link_pose>
+            <use_pose_vector_msg>true</use_pose_vector_msg>
+        </plugin>
     </gazebo>
     <gazebo reference="caster_wheel">
